File: pcb/qTouchTest2.kicad_pcb (KiCad board)
At the start: 2 copper layers, 68.5 x 47 mm, 40 parts, among them CON1 AVR-ISP-6, J1 USB-MINI-B, K1 CONN_3, P1 CONN_1, P2 CONN_1, P3 CONN_1, P6 CONN_1, P7 CONN_1, P8 CONN_1, P9 CONN_1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

Commit message: saving again... not sure what changed
Parts:
- added L2: FERRITE_BEAD, SM0805, F.Cu at (81.6, 76.8)
- moved C6 2.30 mm to (85.3, 76.8), turned to 0 degrees
Connections:
- C6 pad 1: +5V -> N-0000022
- U2 pad 24: +5V -> N-0000022
Routing:
- net GND: track 95.1 -> 104.7 mm
- net N-0000022: track 0.00 -> 6.50 mm
- net +5V: track 86.7 -> 83.5 mm
